Commit message: Updated description to match realvehicle

File: description/camera.xacro (robot description, xacro)
@@ -4,17 +4,10 @@
         <parent link="chassis"/>
         <child link="camera_link"/>
-        <origin xyz="0.276 0 0.181" rpy="0 0 0"/>
+        <origin xyz="0.300 0 0.090" rpy="0 0 0"/>
     </joint>
     <link name="camera_link">
         <visual>
             <geometry>
-                <box size="0.010 0.03 0.03"/>
-            </geometry>
-            <material name="black"/>
-        </visual>
-        <visual>
-            <origin xyz="0 0 -0.05"/>
-            <geometry>
-                <cylinder radius="0.002" length="0.1"/>
+                <box size="0.035 0.055 0.045"/>
             </geometry>
             <material name="black"/>

File: description/lidar.xacro (robot description, xacro)
@@ -4,17 +4,10 @@
         <parent link="chassis"/>
         <child link="laser_frame"/>
-        <origin xyz="0.122 0 0.212" rpy="0 0 0"/>
+        <origin xyz="0.140 0 0.130" rpy="0 0 0"/>
     </joint>
     <link name="laser_frame">
         <visual>
             <geometry>
-                <cylinder radius="0.05" length="0.04"/>
-            </geometry>
-            <material name="black"/>
-        </visual>
-        <visual>
-            <origin xyz="0 0 -0.05"/>
-            <geometry>
-                <cylinder radius="0.01" length="0.1"/>
+                <cylinder radius="0.035" length="0.04"/>
             </geometry>
             <material name="black"/>
@@ -22,8 +15,8 @@
         <collision>
             <geometry>
-                <cylinder radius="0.05" length="0.04"/>
+                <cylinder radius="0.035" length="0.04"/>
             </geometry>
         </collision>
-        <xacro:inertial_cylinder mass="0.1" length="0.04" radius="0.05">
+        <xacro:inertial_cylinder mass="0.1" length="0.04" radius="0.035">
             <origin xyz="0 0 0" rpy="0 0 0"/>
         </xacro:inertial_cylinder>
@@ -32,5 +25,5 @@
         <material>Gazebo/Red</material>
         <sensor name="laser" type="ray">
-            <pose> 0 0 0 0 0 0 </pose>
+            <pose> xyz="0 0 0" rpy="0 0 0" </pose>
             <visualize>false</visualize>
             <update_rate>10</update_rate>

File: description/robot_core.xacro (robot description, xacro)
@@ -1,4 +1,5 @@
 <?xml version="1.0"?>
 <robot xmlns:xacro="http://www.ros.org/wiki/xacro">
+    <xacro:property name="chassis_l" value="375"/>
     <xacro:include filename="inertial_macros.xacro"/>
     <material name="white">
@@ -23,11 +24,18 @@
         <parent link="base_link" />
         <child link="chassis"/>
-        <origin xyz="0 0 0"/>
+        <origin xyz="-0.1875 0 0.006"/>
     </joint>
     <link name="chassis">
         <visual>
-            <origin xyz="0 0 0"/>
+            <origin xyz="0.1875 0 0.045"/>
             <geometry>
-                <box size=".375 .225 .090"/>
+                <box size="0.375 .225 .090"/>
+            </geometry>
+            <material name="white"/>
+        </visual>
+        <visual>
+            <origin xyz="0.135 0 0.110"/>
+            <geometry>
+                <box size=".145 .200 .040"/>
             </geometry>
             <material name="white"/>
@@ -99,13 +107,13 @@
     </gazebo>
     <!-- Castor Wheel Link_-->
-    <joint name="castor_wheel_joint" type="continuous">
+    <joint name="castor_wheel_joint" type="fixed">
         <parent link="base_link" />
         <child link="castor_wheel"/>
-        <origin xyz="0.1 0 -0.065"/>
+        <origin xyz="0.1 0 -0.0"/>
     </joint>
     <link name="castor_wheel">
         <visual>
             <geometry>
-                <sphere radius="0.05"/>
+                <sphere radius="0.09"/>
             </geometry>
             <material name="black"/>
@@ -113,8 +121,8 @@
         <collision>
             <geometry>
-                <sphere radius="0.05"/>
+                <sphere radius="0.09"/>
             </geometry>
        </collision>
-        <xacro:inertial_sphere mass="0.1" radius="0.05">
+        <xacro:inertial_sphere mass="0.1" radius="0.09">
             <origin xyz="0 0 0" rpy="0 0 0"/>
         </xacro:inertial_sphere>

File: description/ros2_control.xacro (robot description, xacro)
@@ -37,5 +37,6 @@
             <param name="example_param_hw_stop_duration_sec">3</param>
             <param name="example_param_hw_slowdown">0</param>
-            <param name="hoverboard_port">/dev/ttyUSB1</param>
+<!--            <param name="hoverboard_port">/dev/ttyUSB0</param> -->
+            <param name="hoverboard_port">/dev/serial/by-path/platform-fd500000.pcie-pci-0000:01:00.0-usb-0:1.3.2:1.0-port0</param>
         </hardware>
         <joint name="left_wheel_joint">
