Commit message: Gazebo should run but it does not

File: description/robot.urdf.xacro (robot description, xacro)
@@ -2,3 +2,4 @@
 <robot xmlns:xacro="http://www.ros.org/wiki/xacro"  name="robot">
     <xacro:include filename="robot_core.xacro"/>
+    <xacro:include filename="gazebo_robot.xacro"/>
 </robot>

File: description/robot_core.xacro (robot description, xacro)
@@ -40,4 +40,7 @@
         </xacro:inertial_box>
     </link>
+    <gazebo reference="chassis">
+        <material>Gazebo/White</material>
+    </gazebo>
 <!-- Left Wheel Link_-->
     <joint name="left_wheel_joint" type="continuous">
@@ -62,6 +65,9 @@
             <origin xyz="0 0 0" rpy="0 0 0"/>
         </xacro:inertial_cylinder>
-</link>
-<!-- Right Wheel Link_-->
+    </link>
+    <gazebo reference="left_wheel">
+        <material>Gazebo/Blue</material>
+    </gazebo>
+    <!-- Right Wheel Link_-->
     <joint name="right_wheel_joint" type="continuous">
         <parent link="base_link" />
@@ -86,5 +92,8 @@
         </xacro:inertial_cylinder>
     </link>
-<!-- Castor Wheel Link_-->
+    <gazebo reference="right_wheel">
+        <material>Gazebo/Blue</material>
+    </gazebo>
+    <!-- Castor Wheel Link_-->
     <joint name="castor_wheel_joint" type="continuous">
         <parent link="base_link" />
@@ -107,4 +116,9 @@
             <origin xyz="0 0 0" rpy="0 0 0"/>
         </xacro:inertial_sphere>
-</link>
+    </link>
+    <gazebo reference="castor_wheel">
+        <material>Gazebo/Black</material>
+        <mu1 value="0.001"/>
+        <mu2 value="0.001"/>
+    </gazebo>
 </robot>

Commit message: Added camera driver

File: description/robot.urdf.xacro (robot description, xacro)
@@ -3,4 +3,5 @@
     <xacro:include filename="robot_core.xacro"/>
 <!--     <xacro:include filename="gazebo_control.xacro"/> -->
+    <xacro:include filename="camera.xacro"/>
     <xacro:include filename="ros2_control.xacro"/>
 </robot>

File: description/robot_core.xacro (robot description, xacro)
@@ -53,5 +53,5 @@
         <visual>
             <geometry>
-                <cylinder radius="0.09" length="0.075"/>
+                <cylinder radius="0.09" length="0.066"/>
             </geometry>
             <material name="blue"/>
@@ -59,5 +59,5 @@
         <collision>
             <geometry>
-                <cylinder radius="0.09" length="0.075"/>
+                <cylinder radius="0.09" length="0.066"/>
             </geometry>
        </collision>
@@ -79,5 +79,5 @@
         <visual>
             <geometry>
-                <cylinder radius="0.09" length="0.075"/>
+                <cylinder radius="0.09" length="0.066"/>
             </geometry>
             <material name="blue"/>
@@ -85,5 +85,5 @@
         <collision>
             <geometry>
-                <cylinder radius="0.09" length="0.075"/>
+                <cylinder radius="0.09" length="0.066"/>
             </geometry>
        </collision>

Commit message: Added Lidar

File: description/robot.urdf.xacro (robot description, xacro)
@@ -4,4 +4,5 @@
 <!--     <xacro:include filename="gazebo_control.xacro"/> -->
     <xacro:include filename="camera.xacro"/>
+    <xacro:include filename="lidar.xacro"/>
     <xacro:include filename="ros2_control.xacro"/>
 </robot>

File: description/robot_core.xacro (robot description, xacro)
@@ -13,4 +13,7 @@
     <material name="black">
         <color rgba="0 0 0 1"/>
+    </material>
+   <material name="red">
+        <color rgba="1 0 0 1"/>
     </material>
 <!-- Base Link_-->

Commit message: Playing with description

File: description/robot.urdf.xacro (robot description, xacro)
@@ -1,6 +1,13 @@
 <?xml version="1.0"?>
 <robot xmlns:xacro="http://www.ros.org/wiki/xacro"  name="robot">
+    <xacro:arg name="use_ros2_control" default="true"/>
+    <xacro:arg name="sim_mode" default="false"/>
     <xacro:include filename="robot_core.xacro"/>
-<!--     <xacro:include filename="gazebo_control.xacro"/> -->
+    <xacro:if value="$(arg use_ros2_control)">
+        <xacro:include filename="ros2_control.xacro" />
+    </xacro:if>
+    <xacro:unless value="$(arg use_ros2_control)">
+        <xacro:include filename="gazebo_control.xacro" />
+    </xacro:unless>
     <xacro:include filename="camera.xacro"/>
     <xacro:include filename="lidar.xacro"/>

File: description/robot_core.xacro (robot description, xacro)
@@ -1,6 +1,6 @@
 <?xml version="1.0"?>
 <robot xmlns:xacro="http://www.ros.org/wiki/xacro">
-    <xacro:property name="chassis_l" value="375"/>
     <xacro:include filename="inertial_macros.xacro"/>
+    <xacro:property name="chassis_l" value="0.375"/>
     <material name="white">
         <color rgba="1 1 1 1"/>

File: description/ros2_control.xacro (robot description, xacro)
@@ -28,9 +28,4 @@
 <!--             <param name="left_wheel_name">left_wheel_joint</param>
             <param name="right_wheel_name">right_wheel_joint</param>
-            <param name="loop_rate">30</param>
-            <param name="device">/dev/ttyUSB0</param>
-            <param name="baud_rate">57600</param>
-            <param name="timeout">1000</param>
-            <param name="enc_counts_per_rev">3436</param>
  -->
             <param name="example_param_hw_start_duration_sec">0</param>
