Commit message: Add parameters for SLAM

File: description/robot_core.xacro (robot description, xacro)
@@ -18,7 +18,16 @@
         <color rgba="1 0 0 1"/>
     </material>
-<!-- Base Link_-->
+    <!-- Base Link_-->
     <link name="base_link">
     </link>
+    <!-- Base footprint link -->
+    <joint name="base_footprint_joint" type="fixed">
+        <parent link="base_link" />
+        <child link="base_footprint"/>
+        <origin xyz="0 0 0" rpy="0 0 0"/>
+    </joint>
+    <link name="base_footprint">
+    </link>
+    <!-- Chassis link -->
     <joint name="chassis_joint" type="fixed">
         <parent link="base_link" />
